File: Embedded/Embedded.kicad_sch (KiCad schematic)
At the start: 63 parts, among them J1 GyroBreakout, J2 Conn_01x08, J3 Conn_01x08, J6 Conn_01x08, J7 Conn_01x08, SW1 BackboardSw, U1 ESP32-C6-WROOM-1, U2 BQ25895RTW, U3 FSUSB30MUX, U5 MP8715, U7 SN74AHCT125N, U8 SN74AHCT125N

Commit message: small changes, big dreams
Parts:
- removed C17: 10uF, Capacitor_SMD:C_0603_1608Metric_Pad1.08x0.95mm_HandSolder, symbol Device:C
- added D1, D2: 1N5819, Diode_THT:D_DO-41_SOD81_P10.16mm_Horizontal, symbol Diode:1N5819
- added M1: Fan, Capacitor_SMD:C_1808_4520Metric_Pad1.72x2.30mm_HandSolder, symbol Motor:Fan
- added Q1: FQP27P06, Package_TO_SOT_THT:TO-220-3_Vertical, symbol Transistor_FET:FQP27P06
Connections:
- net +5V: now also D1.1 (K), M1.1 (+)
- net GND: now also D2.2 (A), Q1.2 (D)
- net at C1.1, H12.1, U2.1 (VBUS): now also D2.1 (K)
- net at J1.3 (Pin_3): now also U1.24 (U0RXD/GPIO17)
- net at J3.4 (Pin_4): now also U7.11 (4Y); no longer U7.3 (1Y)
- net at J3.5 (Pin_5): now also U7.8 (3Y); no longer U7.6 (2Y)
- net at J3.6 (Pin_6): now also U7.6 (2Y); no longer U7.8 (3Y)
- net at J3.7 (Pin_7): now also U7.3 (1Y); no longer U7.11 (4Y)
- net at U1.25 (U0TXD/GPIO16): now also Q1.1 (G)
- new net: D1.2 (A), M1.2 (-), Q1.3 (S)
- no-connect marks 22 -> 19
Other:
- note added: "Ambient light sensor read"
- note added: "BMS Charge Enable"
- note added: "BMS Int"
- note added: "BMS OTG"
- note added: "Backboard Button"
- note added: "Base Res Measurement"
- note added: "Buck Power OK"
- note added: "DFPlayer TX"
- note added: "EN"
- note added: "ESP32 USB D+"
- note added: "ESP32 USB D-"
- note added: "Gyro/Inclinometer Int"
- note added: "Helix Neo SIG"
- note added: "Internal Fan Control"
- note added: "MUX S0"
- note added: "MUX S1"
- note added: "MUX S2"
- note added: "MUX S3"
- note added: "Neo MUX EN"
- note added: "Neo MUX S0"
- note added: "Neo MUX S1"
- note added: "Neo MUX S2"
- note added: "Neo MUX S3"
- note added: "Neo MUX SIG"
- note added: "NeoPixel SIG"
- note added: "Res MUX EN"
- note added: "SCL"
- note added: "SDA"
- note added: "Touch button read"
- note added: "USB D+"
- note added: "USB D-"
- note added: "USB MUX Dev Sel"
- note added: "USB MUX Device Select"
- moved on the sheet: J6, J7, R3

Commit message: Old model, new connectors
Parts:
- removed ALS1, H9, Neo3, Touch3: GND, Connector_Wire:SolderWirePad_1x01_SMD_1.5x3mm, symbol Mechanical:MountingHole_Pad
- removed ALS2, Neo2, Touch2: SIG, Connector_Wire:SolderWirePad_1x01_SMD_1.5x3mm, symbol Mechanical:MountingHole_Pad
- removed ALS3, H12, Neo1, Touch1: VCC, Connector_Wire:SolderWirePad_1x01_SMD_1.5x3mm, symbol Mechanical:MountingHole_Pad
- removed H10: CC1, Connector_Wire:SolderWirePad_1x01_SMD_1.5x3mm, symbol Mechanical:MountingHole_Pad
- removed H11: CC2, Connector_Wire:SolderWirePad_1x01_SMD_1.5x3mm, symbol Mechanical:MountingHole_Pad
- removed H7: D-, Connector_Wire:SolderWirePad_1x01_SMD_1.5x3mm, symbol Mechanical:MountingHole_Pad
- removed H8: D+, Connector_Wire:SolderWirePad_1x01_SMD_1.5x3mm, symbol Mechanical:MountingHole_Pad
- removed LS1: Speaker, Capacitor_SMD:C_1808_4520Metric_Pad1.72x2.30mm_HandSolder, symbol Device:Speaker
- removed M1: Fan, Capacitor_SMD:C_1808_4520Metric_Pad1.72x2.30mm_HandSolder, symbol Motor:Fan
- added C17: 100nF, Capacitor_SMD:C_0402_1005Metric_Pad0.74x0.62mm_HandSolder, symbol Device:C
- added C18: 1uF, Capacitor_SMD:C_0603_1608Metric_Pad1.08x0.95mm_HandSolder, symbol Device:C
- added J10: TouchButton, Connector_PinHeader_2.54mm:PinHeader_1x03_P2.54mm_Horizontal, symbol Connector_Generic:Conn_01x03
- added J11: USB-C Breakout, Connector_PinHeader_2.54mm:PinHeader_1x06_P2.54mm_Horizontal, symbol Connector_Generic:Conn_01x06
- added J4: HelixNeo, Connector_PinHeader_2.54mm:PinHeader_1x03_P2.54mm_Horizontal, symbol Connector_Generic:Conn_01x03
- added J5: FanConnector, Connector_PinHeader_2.54mm:PinHeader_1x02_P2.54mm_Horizontal, symbol Connector_Generic:Conn_01x02
- added J8: Speaker, Connector_PinHeader_2.54mm:PinHeader_1x02_P2.54mm_Horizontal, symbol Connector_Generic:Conn_01x02
- added J9: LightSensor, Connector_PinHeader_2.54mm:PinHeader_1x03_P2.54mm_Horizontal, symbol Connector_Generic:Conn_01x03
- added R14: 10k, Resistor_THT:R_Axial_DIN0207_L6.3mm_D2.5mm_P10.16mm_Horizontal, symbol Device:R
- added SW2: BackboardSw, Button_Switch_THT:SW_PUSH_6mm_H5mm, symbol Switch:SW_Push
- C1: footprint Capacitor_SMD:C_0603_1608Metric_Pad1.08x0.95mm_HandSolder -> Capacitor_SMD:C_0402_1005Metric_Pad0.74x0.62mm_HandSolder
- C13: value 10nF -> 100nF
- J2: value Conn_01x08 -> BaseResMUX
- J3: value Conn_01x08 -> BaseNeoMUX
- R13: value 4.7k -> 10k
Connections:
- net +3.3V: now also J10.1 (Pin_1), J9.1 (Pin_1), R14.2
- net +5V: now also J4.1 (Pin_1), J5.1 (Pin_1)
- net GND: now also C18.1, J10.3 (Pin_3), J11.1 (Pin_1), J4.3 (Pin_3), J8.2 (Pin_2), J9.3 (Pin_3)
- net Battery: now reaches BT1.1 (+), BT2.1 (+), C8.1, U2.13 (BAT), U2.14 (BAT)
- net SCL: now reaches J1.8 (Pin_8), R11.2, U1.21 (GPIO23), U2.5 (SCL)
- net FanOut: now reaches D1.2 (A), Q1.3 (S)
- net FanOut: now also J5.2 (Pin_2)
- net at R1.1: now also J11.5 (Pin_5)
- net BaseNeoEN: now reaches U1.23 (GPIO15), U8.2 (1A)
- net BaseNeoSIG: now reaches U1.17 (GPIO19), U8.5 (2A)
- net HelixNeo: now reaches U8.8 (3Y)
- net HelixNeo: now also J4.2 (Pin_2)
- net HelixNeoSIG: now reaches U1.18 (GPIO20), U8.9 (3A)
- net BuckPOK: now reaches R10.1, U1.26 (GPIO3/ADC1_CH3), U5.6 (POK)
- net BackboardIcBtn: now reaches D3.1, U2.12 (~{QON})
- net BackboardBtn: now reaches D3.2
- net BackboardBtn: now also U1.7 (MTDO/GPIO7); no longer U1.6 (MTCK/GPIO6/ADC1_CH6)
- net UsbD-: now reaches U3.6 (D-)
- net UsbD-: now also J11.3 (Pin_3)
- net Spk+: now reaches J6.6 (Pin_6)
- net Spk+: now also J8.1 (Pin_1)
- net UsbVBUS: now reaches C1.1, D2.1 (K), U2.1 (VBUS)
- net UsbVBUS: now also J11.2 (Pin_2)
- net UsbDSEL: now reaches R3.1, U2.24 (DSEL), U3.1 (S)
- net SDA: now reaches J1.7 (Pin_7), R12.2, U1.20 (GPIO22), U2.6 (SDA)
- net BmsInt: now reaches U2.7 (~{INT})
- net BmsInt: now also U1.6 (MTCK/GPIO6/ADC1_CH6); no longer U1.5 (MTDI/GPIO5/ADC1_CH5)
- net BmsOTG: now reaches U1.19 (GPIO21), U2.8 (OTG)
- net BmsCE: now reaches U2.9 (~{CE})
- net BmsCE: now also U1.25 (U0TXD/GPIO16); no longer U1.4 (MTMS/GPIO4/ADC1_CH4)
- net BaseResSIG: now reaches J2.8 (Pin_8), R13.2, U1.8 (GPIO0/ADC1_CH0/XTAL_32K_P)
- net EspD+: now reaches U1.14 (GPIO13/USB_D+), U3.3 (HSD2+)
- net UsbD+: now reaches U3.4 (D+)
- net UsbD+: now also J11.4 (Pin_4)
- net EspD-: now reaches U1.13 (GPIO12/USB_D-), U3.7 (HSD2-)
- net ALS: now reaches U1.9 (GPIO1/ADC1_CH1/XTAL_32K_N)
- net ALS: now also J9.2 (Pin_2)
- net GyroInt: now reaches J1.3 (Pin_3), U1.24 (U0RXD/GPIO17)
- net DFPlayer: now reaches J6.2 (Pin_2)
- net DFPlayer: now also U1.5 (MTDI/GPIO5/ADC1_CH5); no longer U1.7 (MTDO/GPIO7)
- net FanControl: now reaches Q1.1 (G)
- net FanControl: now also U1.4 (MTMS/GPIO4/ADC1_CH4); no longer U1.25 (U0TXD/GPIO16)
- net at R2.1: now also J11.6 (Pin_6)
- net BaseNeoS0: now reaches J3.4 (Pin_4), U7.11 (4Y)
- net BaseNeoS1: now reaches J3.5 (Pin_5), U7.8 (3Y)
- net BaseNeoS2: now reaches J3.6 (Pin_6), U7.6 (2Y)
- net BaseNeoS3: now reaches J3.7 (Pin_7), U7.3 (1Y)
- net TouchBtn: now reaches U1.27 (GPIO2/ADC1_CH2)
- net TouchBtn: now also J10.2 (Pin_2)
- net BaseResEN: now reaches J2.3 (Pin_3), U1.16 (GPIO18)
- net MuxS0: now reaches J2.4 (Pin_4), U1.12 (GPIO11), U7.12 (4A)
- net MuxS1: now reaches J2.5 (Pin_5), U1.11 (GPIO10), U7.9 (3A)
- net MuxS2: now reaches J2.6 (Pin_6), U1.15 (GPIO9), U7.5 (2A)
- net MuxS3: now reaches J2.7 (Pin_7), U1.10 (GPIO8), U7.2 (1A)
- net at U1.3 (EN/CHIP_PU): now also C17.1, C18.2, SW2.1
- new net Esp32EN: C17.2, R14.1, SW2.2
- no-connect marks 19 -> 18
Other:
- note removed: "Ambient light sensor"
- note removed: "Ambient light sensor read"
- note removed: "BMS Charge Enable"
- note removed: "BMS OTG"
- note removed: "Backboard Button"
- note removed: "Base Res Measurement"
- note removed: "DFPlayer TX"
- note removed: "EN"
- note removed: "ESP32 USB D+"
- note removed: "ESP32 USB D-"
- note removed: "Gyro/Inclinometer Int"
- note removed: "Helix Neo SIG"
- note removed: "Helix NeoPixels"
- note removed: "Internal Fan Control"
- note removed: "Neo MUX EN"
- note removed: "Neo MUX S0"
- note removed: "Neo MUX S1"
- note removed: "Neo MUX S2"
- note removed: "Neo MUX S3"
- note removed: "Neo MUX SIG"
- note removed: "NeoPixel SIG"
- note removed: "Res MUX EN"
- note removed: "Touch button"
- note removed: "Touch button read"
- note removed: "USB D+"
- note removed: "USB D-"
- note removed: "USB MUX Dev Sel"
- note removed: "USB MUX Device Select"
- note removed: "USB breakout board pads"
- moved on the sheet: BT1, BT2, C8, R1, R13, R2

Commit message: v4
Parts:
- added BT3, BT4: Battery_Cell, Connector_JST:JST_PH_B2B-PH-K_1x02_P2.00mm_Vertical, symbol Device:Battery_Cell
- added F1, F2, F3, F4: Polyfuse, Fuse:Fuse_1206_3216Metric_Pad1.42x1.75mm_HandSolder, symbol Device:Polyfuse
- added Q2, Q4, Q6, Q8: FS8205A, Package_SO:MSOP-8_3x3mm_P0.65mm, symbol symbols:FS8205A
- added Q3, Q5, Q7, Q9: AO3401A, Package_TO_SOT_SMD:TSOT-23_HandSoldering, symbol Transistor_FET:AO3401A
- added R15, R16, R17, R18, R19, R20, R21, R22: 100, Resistor_THT:R_Axial_DIN0207_L6.3mm_D2.5mm_P10.16mm_Horizontal, symbol Device:R
- added U10, U4, U6, U9: DW01A, Package_TO_SOT_SMD:SOT-23-6, symbol Battery_Management:DW01A
- BT1, BT2: footprint Capacitor_SMD:C_1808_4520Metric_Pad1.72x2.30mm_HandSolder -> Connector_JST:JST_PH_B2B-PH-K_1x02_P2.00mm_Vertical
- Q1: footprint Package_TO_SOT_THT:TO-220-3_Vertical -> Package_TO_SOT_THT:TO-220-3_Horizontal_TabDown
Connections:
- net GND: now also C8.1, Q2.2 (S1_1), Q2.3 (S1_2), Q4.2 (S1_1), Q4.3 (S1_2), Q6.2 (S1_1), Q6.3 (S1_2), Q8.2 (S1_1), Q8.3 (S1_2), R16.1, R18.1, R20.1, R22.1; no longer BT1.2 (-), BT2.2 (-), C8.2
- removed net Battery: BT1.1 (+), BT2.1 (+), C8.1, U2.13 (BAT), U2.14 (BAT)
- new net: R18.2, U6.2 (CS)
- new net: Q6.1 (D12_1), Q6.8 (D12_2)
- new net: Q6.4 (G1), U9.1 (OD)
- new net: Q6.5 (G2), U9.3 (OC)
- new net: BT3.2 (-), Q6.6 (S2_1), Q6.7 (S2_2), Q7.1 (G), U9.6 (GND)
- new net: R20.2, U9.2 (CS)
- new net: R19.1, U9.5 (VCC)
- new net: BT2.1 (+), Q5.2 (S)
- new net: BT2.2 (-), Q4.6 (S2_1), Q4.7 (S2_2), Q5.1 (G), U6.6 (GND)
- new net: Q4.1 (D12_1), Q4.8 (D12_2)
- new net: Q4.4 (G1), U6.1 (OD)
- new net: Q4.5 (G2), U6.3 (OC)
- new net: R16.2, U4.2 (CS)
- new net: BT4.2 (-), Q8.6 (S2_1), Q8.7 (S2_2), Q9.1 (G), U10.6 (GND)
- new net: BT4.1 (+), Q9.2 (S)
- new net: F4.2, Q9.3 (D), R21.2
- new net: Q8.4 (G1), U10.1 (OD)
- new net: R22.2, U10.2 (CS)
- new net: Q8.5 (G2), U10.3 (OC)
- new net: R21.1, U10.5 (VCC)
- new net: R17.1, U6.5 (VCC)
- new net: F2.2, Q5.3 (D), R17.2
- new net: Q2.4 (G1), U4.1 (OD)
- new net: Q2.5 (G2), U4.3 (OC)
- new net: R15.1, U4.5 (VCC)
- new net: BT1.2 (-), Q2.6 (S2_1), Q2.7 (S2_2), Q3.1 (G), U4.6 (GND)
- new net: F1.2, Q3.3 (D), R15.2
- new net: BT1.1 (+), Q3.2 (S)
- new net: F3.2, Q7.3 (D), R19.2
- new net: BT3.1 (+), Q7.2 (S)
- new net: Q2.1 (D12_1), Q2.8 (D12_2)
- new net: Q8.1 (D12_1), Q8.8 (D12_2)
- new net BATT: C8.2, F1.1, F2.1, F3.1, F4.1, U2.13 (BAT), U2.14 (BAT)
Other:
- moved on the sheet: C2, C3, C4, C5, C6, C7, C8, D1, J4, J5, Q1

Commit message: Overhaul
Redesign, Ground for UWP/Droid app, Switch from Arduino C to ESP-IDF with native C
Connections:
- net BaseNeoS0: now also U7.6 (2Y); no longer U7.11 (4Y)
- net BaseNeoS2: now also U7.11 (4Y); no longer U7.6 (2Y)
- net MuxS0: now also U7.5 (2A); no longer U7.12 (4A)
- net MuxS2: now also U7.12 (4A); no longer U7.5 (2A)
Changed lines of the file:
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@@
 	(wire
 		(pts
-			(xy 168.91 48.26) (xy 168.91 54.61)
-		)
-		(stroke
-			(width 0)
-			(type default)
-		)
-	)
-	(wire
-		(pts
 			(xy 59.69 185.42) (xy 59.69 191.77)
 		)
@@
 	(wire
 		(pts
-			(xy 114.3 35.56) (xy 132.08 35.56)
-		)
-		(stroke
-			(width 0)
-			(type default)
-		)
-	)
-	(wire
-		(pts
 			(xy 279.4 139.7) (xy 279.4 146.05)
 		)
@@
 	(wire
 		(pts
-			(xy 171.45 59.69) (xy 184.15 59.69)
+			(xy 168.91 48.26) (xy 168.91 59.69)
 		)
 		(stroke
@@
 	(wire
 		(pts
-			(xy 168.91 54.61) (xy 184.15 54.61)
+			(xy 255.27 97.79) (xy 257.81 97.79)
 		)
 		(stroke
@@
 	(wire
 		(pts
-			(xy 255.27 97.79) (xy 257.81 97.79)
+			(xy 116.84 77.47) (xy 132.08 77.47)
 		)
 		(stroke
@@
 	(wire
 		(pts
-			(xy 116.84 77.47) (xy 132.08 77.47)
+			(xy 234.95 129.54) (xy 219.71 129.54)
 		)
 		(stroke
@@
 	(wire
 		(pts
-			(xy 234.95 129.54) (xy 219.71 129.54)
+			(xy 226.06 123.19) (xy 226.06 124.46)
 		)
 		(stroke
@@
 	(wire
 		(pts
-			(xy 226.06 123.19) (xy 226.06 124.46)
+			(xy 254 20.32) (xy 254 17.78)
 		)
 		(stroke
@@
 	(wire
 		(pts
-			(xy 254 20.32) (xy 254 17.78)
+			(xy 63.5 185.42) (xy 59.69 185.42)
 		)
 		(stroke
@@
 	(wire
 		(pts
-			(xy 63.5 185.42) (xy 59.69 185.42)
+			(xy 168.91 59.69) (xy 184.15 59.69)
 		)
 		(stroke
@@
 	(wire
 		(pts
+			(xy 114.3 50.8) (xy 132.08 50.8)
+		)
+		(stroke
+			(width 0)
+			(type default)
+		)
+	)
+	(wire
+		(pts
 			(xy 16.51 154.94) (xy 39.37 154.94)
 		)
@@
 	(wire
 		(pts
-			(xy 171.45 33.02) (xy 171.45 59.69)
+			(xy 171.45 33.02) (xy 171.45 54.61)
 		)
 		(stroke
@@
 	(wire
 		(pts
+			(xy 171.45 54.61) (xy 184.15 54.61)
+		)
+		(stroke
+			(width 0)
+			(type default)
+		)
+	)
+	(wire
+		(pts
 			(xy 223.52 16.51) (xy 223.52 20.32)
 		)
@@
 	(wire
 		(pts
-			(xy 116.84 66.04) (xy 116.84 50.8)
+			(xy 116.84 35.56) (xy 116.84 66.04)
 		)
 		(stroke
@@
 	(wire
 		(pts
-			(xy 93.98 58.42) (xy 107.95 58.42)
+			(xy 116.84 35.56) (xy 132.08 35.56)
 		)
 		(stroke
@@
 	(wire
 		(pts
-			(xy 252.73 128.27) (xy 247.65 128.27)
+			(xy 93.98 58.42) (xy 107.95 58.42)
 		)
 		(stroke
@@
 	(wire
 		(pts
-			(xy 115.57 76.2) (xy 93.98 76.2)
+			(xy 252.73 128.27) (xy 247.65 128.27)
 		)
 		(stroke
@@
 	(wire
 		(pts
-			(xy 93.98 60.96) (xy 109.22 60.96)
+			(xy 115.57 76.2) (xy 93.98 76.2)
 		)
 		(stroke
@@
 	(wire
 		(pts
-			(xy 99.06 106.68) (xy 99.06 83.82)
+			(xy 93.98 60.96) (xy 109.22 60.96)
 		)
 		(stroke
@@
 	(wire
 		(pts
-			(xy 222.25 25.4) (xy 223.52 25.4)
+			(xy 99.06 106.68) (xy 99.06 83.82)
 		)
 		(stroke
@@
 	(wire
 		(pts
-			(xy 102.87 113.03) (xy 102.87 78.74)
+			(xy 222.25 25.4) (xy 223.52 25.4)
 		)
 		(stroke
@@
 	(wire
 		(pts
-			(xy 116.84 50.8) (xy 132.08 50.8)
+			(xy 102.87 113.03) (xy 102.87 78.74)
 		)
 		(stroke
@@
 	(wire
 		(pts
-			(xy 114.3 60.96) (xy 114.3 35.56)
+			(xy 114.3 60.96) (xy 114.3 50.8)
 		)
 		(stroke
@@
 		)
 	)
-	(label "BaseNeoS0"
+	(label "BaseNeoS2"
 		(at 168.91 48.26 180)
 		(effects
@@
 		)
 	)
-	(label "BaseNeoS2"
+	(label "BaseNeoS0"
 		(at 170.18 33.02 180)
 		(effects
